File: Saab_Rear_LED_Enabler.kicad_sch (KiCad schematic)
At the start: 47 parts, among them J2 Conn_01x12_Pin, U1 ESP32-DEVKIT-V1, U3 MAX11611EEET, U9 NCP1117ST50T3G

Commit message: LED Enabler updated to v0.80, see Changelog for details
Parts:
- added C3, C4: 0.1u, Capacitor_SMD:C_0603_1608Metric, symbol Device:C_Small
- added R36: 2k, Resistor_SMD:R_0402_1005Metric_Pad0.72x0.64mm_HandSolder, symbol Device:R_US
- R1, R2: footprint (none) -> Resistor_SMD:R_0805_2012Metric
- U1: footprint ESP32-DEVKIT-V1:MODULE_ESP32_DEVKIT_V1 -> czabel_personal:ESP32_DEVKIT_V1_30PIN
- U3: footprint MAX11611EEET:SOP63P602X175-16N -> czabel_personal:SOP63P602X175-16N
Connections:
- net GND: now also C3.2, C4.2
- net 3V3: now reaches R1.1, R2.1, U1.1 (3V3), U3.16 (VDD)
- net 3V3: now also C3.1
- net SCL: now reaches R2.2, U1.14 (D22), U3.13 (SCL)
- net SDA: now reaches R1.2, U1.11 (D21), U3.14 (SDA)
- net 5V: now reaches C2.1, U1.30 (VIN), U9.2 (OUT)
- net at U3.1 (AIN11/REF): now also R36.1
- new net: C4.1, R36.2
Other:
- moved on the sheet: R10, R11, R12, R13, R14, R15, R16, R17, R3, R4, R5, R6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
